Commit message: 🚧 引入SJTU机器人学库

File: model/miniArm_URDF/urdf/miniarm.urdf (robot description, URDF)
Before this commit: robot mini1, 7 links, 6 joints
Joints:
- joint joint3: origin xyz=0.14 0 0.01245 rpy=3.1416 0 0 -> xyz=0.14 0 0.01245 rpy=3.1416 0 -1.5708
- joint joint4: origin xyz=0 0.012 0.054 rpy=1.5708 0 0 -> xyz=0 0.012 0.054 rpy=1.5708 0 3.1416

File: model/miniArm_URDF/urdf/miniarm_collision_test.urdf (robot description, URDF)
Before this commit: robot mini1_collision_test, 7 links, 6 joints
Joints:
- joint joint3: limit lower=-0.785398 upper=1.1570796 effort=9.0 velocity=18.0 -> lower=-2.7925 upper=0.0 effort=9.0 velocity=18.0; origin xyz=0.14 0 0.01245 rpy=3.1416 0 0 -> xyz=0.14 0 0.01245 rpy=3.1416 0 -1.5708
- joint joint4: limit lower=-3.1415926535 upper=3.1415926535 effort=3.5 velocity=18.0 -> lower=-1.5708 upper=1.5708 effort=3.5 velocity=18.0; origin xyz=0 0.012 0.054 rpy=1.5708 0 0 -> xyz=0 0.012 0.054 rpy=1.5708 3.1415 0
